File: T17_Schematic_The_Useless_Box.brd (EAGLE design)
At the start: 100 x 80 mm, 18 parts, among them U1 ATMEGA328P-AU

Commit message: Circuit rev...? board rev 1
Parts:
- removed S1: (no value), switch:REKN
- added S2: SWITCH-MOMENTARY-2SMD, SparkFun-Electromechanical:TACTILE-SWITCH-SMD
Connections:
- removed net AVCC: U1.18
- removed net N$13: U1.15
- removed net N$15: MOTOR_DRIVER_1.2, MOTOR_DRIVER_1.3
- removed net N$17: MOTOR_DRIVER_2.2, MOTOR_DRIVER_2.3
- removed net N$28: S1.1A, S1.1B
- net +5V: now also MOTOR_DRIVER_1.2, MOTOR_DRIVER_1.3, MOTOR_DRIVER_2.2, MOTOR_DRIVER_2.3, U1.18
- net GND: now also S2.1; no longer S1.0A, S1.0B
- net N$12: now also S2.3
- net N$9: now also U1.15
Routing:
- net +5V: track 54.8 -> 129.0 mm, vias 0 -> 3
- net N$12: track 13.0 -> 66.3 mm, vias 0 -> 2
- net N$23: track 0.00 -> 35.3 mm, vias 0 -> 1
- net N$9: track 0.00 -> 32.0 mm, vias 0 -> 1
- net N$22: track 0.00 -> 28.4 mm, vias 0 -> 1
- net N$11: track 0.00 -> 25.5 mm, vias 0 -> 2
- net N$14: track 0.00 -> 25.3 mm, vias 0 -> 2
- net N$28: track 10.2 -> 0.00 mm
- net N$8: track 34.7 -> 41.0 mm
- net GND: track 208.8 -> 214.0 mm, vias 1 -> 6
- net N$17: track 1.27 -> 0.00 mm
- net N$15: track 1.27 -> 0.00 mm
- net N$19: track 29.6 -> 30.5 mm
