File: T17_Schematic_The_Useless_Box.sch (EAGLE design)
At the start: 21 parts, among them IC1 AT89S51-24P, X1 22-23-2021, X2 22-23-2021

Commit message: Added Latest Version of the schematic and the board
Parts:
- removed 5V_VOLTAGE_REGULATOR: (no value), v-reg:78LXX
- removed 9V_BATTERY: AB9V, battery:AB9V
- removed LED: LAP4-TOP, led:LAP4-TOP
- removed R1: 10k, rcl:R-EU_R0805
- removed R4: 0, rcl:R-EU_R0805
- removed X1, X2: 22-23-2021, con-molex:22-23-2021
- added DC_MOTOR_1, DC_MOTOR_2: 22-23-2021, con-molex:22-23-2021
- added G1: AB9V, battery:AB9V
- added U1: ATMEGA328P-AU, Atmel_By_element14_Batch_1-00:ATMEGA328P-AU
- C1, C2: value 22p -> 10uF
- C3, C4: value 10n -> 10nF
- IC1: value AT89S51-24P -> (none); device atmel:AT89S51-24P -> v-reg:78LXX
- R2: value 1k -> 0
- R3: value 10 -> 10k
Connections:
- removed net N$10: IC1G$1.P0.1_AD1
- removed net N$16: R3.1, R4.2
- removed net N$2: IC1G$1.P1.7_SCK, ICSP.3, R2.2
- removed net N$4: MOTOR_DRIVER_1.OUT1, X1-1.S
- removed net N$5: IC1G$1.P1.5_MOSI, ICSP.4, S1.0@A, S1.0@B
- removed net VCC: R1.1
- new net +5V: ARM_SERVO.1, C1.1, IC1.OUT, ICSP.2, LID_SERVO.1, R3.2, U1.VCC, U1.VCC_2
- new net N$26: DC_MOTOR_1-2.S, MOTOR_DRIVER_1.OUT2
- new net N$27: DC_MOTOR_2-2.S, MOTOR_DRIVER_2.OUT2
- new net N$28: S1.1@A, S1.1@B
- net GND: now also C1.2, C2.2, C3.2, C4.2, G1.-, IC1.GND, S1.0@A, S1.0@B, U1.GND, U1.GND_2, U1.GND_3; no longer 5V_VOLTAGE_REGULATOR.GND, 9V_BATTERY.-, C1.1, C2.1, LED.C, S1.1@A, S1.1@B
- net N$1: now also ICSP.3, U1.PB5; no longer IC1G$1.P1.6_MISO, ICSP.1
- net N$11: now also C3.1, U1.PB6; no longer LED.A, R2.1
- net N$12: now also ICSP.5, R3.1, U1.PC6; no longer 5V_VOLTAGE_REGULATOR.OUT, C3.1
- net N$13: now also U1.PB3; no longer 5V_VOLTAGE_REGULATOR.IN, C4.2
- net N$14: now also U1.PB7; no longer SCHMIDT_TRIGGER.C
- net N$15: now also MOTOR_DRIVER_1.VCC@1, MOTOR_DRIVER_1.VCC@2; no longer R3.2, SCHMIDT_TRIGGER.A
- net N$17: now also MOTOR_DRIVER_2.VCC@1, MOTOR_DRIVER_2.VCC@2; no longer 9V_BATTERY.+, R4.1
- net N$18: now also MOTOR_DRIVER_1.FIN, U1.PC3; no longer MOTOR_DRIVER_2.GND
- net N$19: now also MOTOR_DRIVER_1.RIN, U1.PC2; no longer IC1G$1.P0.2_AD2, MOTOR_DRIVER_1.FIN
- net N$20: now also MOTOR_DRIVER_2.FIN, U1.PC5; no longer IC1G$1.P0.3_AD3, MOTOR_DRIVER_1.RIN
- net N$21: now also MOTOR_DRIVER_2.RIN, U1.PC4; no longer IC1G$1.P0.4_AD4, MOTOR_DRIVER_2.FIN
- net N$22: now also LID_SERVO.2, U1.PC0; no longer IC1G$1.P0.5_AD5, MOTOR_DRIVER_2.RIN
- net N$23: now also ARM_SERVO.2, U1.PC1; no longer MOTOR_DRIVER_1.OUT2, X1-2.S
- net N$24: now also DC_MOTOR_2-1.S; no longer X2-1.S
- net N$25: now also DC_MOTOR_1-1.S, MOTOR_DRIVER_1.OUT1; no longer MOTOR_DRIVER_2.OUT2, X2-2.S
- net N$3: now also C2.1, IC1.IN, SCHMIDT_TRIGGER.C; no longer IC1G$1.RST, ICSP.5, R1.2
- net N$6: now also R2.2, SCHMIDT_TRIGGER.A; no longer C1.2, IC1G$1.XTAL1
- net N$7: now also G1.+, R2.1; no longer ARM_SERVO.1, C3.2, IC1G$1.VCC, ICSP.2, LID_SERVO.1, MOTOR_DRIVER_1.VCC@1, MOTOR_DRIVER_1.VCC@2, MOTOR_DRIVER_2.VCC@1, MOTOR_DRIVER_2.VCC@2
- net N$8: now also ICSP.1, U1.PB4; no longer IC1G$1.P0.0_AD0, LID_SERVO.2
- net N$9: now also ICSP.4; no longer C2.2, IC1G$1.XTAL2
Other:
- note added: "ATMega328"
- note added: "DC MOTORS"
- note added: "MOTOR DRIVERS"
- note added: "POWER SUPPLY"
- note removed: "1"
- note removed: "10/29/2014"
- note removed: "2"
- note removed: "DC Motor 1"
- note removed: "DC Motor 2"
- note removed: "Note: IC1 is a placeholder due to drop incidents. We will be using the ATMega328."
- note removed: "Power Supply"
- note removed: "See Note"
- moved on the sheet: ARM_SERVO, C1, C2, C3, C4, ICSP, LID_SERVO, MOTOR_DRIVER_1, MOTOR_DRIVER_2, R2, R3, S1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

Commit message: Circuit rev...? board rev 1
Parts:
- removed S1: (no value), switch:REKN
- added S2: SWITCH-MOMENTARY-2SMD, SparkFun-Electromechanical:SWITCH-MOMENTARY-2SMD
Connections:
- removed net N$13: U1.PB3
- removed net N$15: MOTOR_DRIVER_1.VCC@1, MOTOR_DRIVER_1.VCC@2
- removed net N$17: MOTOR_DRIVER_2.VCC@1, MOTOR_DRIVER_2.VCC@2
- removed net N$28: S1.1@A, S1.1@B
- net +5V: now also MOTOR_DRIVER_1.VCC@1, MOTOR_DRIVER_1.VCC@2, MOTOR_DRIVER_2.VCC@1, MOTOR_DRIVER_2.VCC@2, U1.AVCC
- net GND: now also S2.1; no longer S1.0@A, S1.0@B
- net N$12: now also S2.2
- net N$9: now also U1.PB3

Commit message: Circuit revision checked, this is rev 2. modified the circuit schematic to reflect as much in the bottom right. Stay tuned for Rev 3.
Other:
- note added: "2"
Changed lines of the file:
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@@
 <setting verticaltext="up"/>
 </settings>
-<grid distance="0.01" unitdist="inch" unit="inch" style="lines" multiple="1" display="yes" altdistance="0.01" altunitdist="inch" altunit="inch"/>
+<grid distance="0.1" unitdist="inch" unit="inch" style="lines" multiple="1" display="no" altdistance="0.01" altunitdist="inch" altunit="inch"/>
 <layers>
 <layer number="1" name="Top" color="4" fill="1" visible="no" active="no"/>
@@
 <wire x1="419.1" y1="-121.92" x2="382.27" y2="-121.92" width="0.1524" layer="97"/>
 <text x="393.7" y="-162.56" size="1.778" layer="90">DC MOTORS</text>
+<text x="419.1" y="-236.22" size="1.778" layer="91">2</text>
 </plain>
 <instances>
@@
 <net name="N$20" class="0">
 <segment>
-<wire x1="264.16" y1="-73.66" x2="264.16" y2="-76.454" width="0.1524" layer="91"/>
 <pinref part="MOTOR_DRIVER_2" gate="P" pin="FIN"/>
 <wire x1="264.16" y1="-76.454" x2="264.16" y2="-193.04" width="0.1524" layer="91"/>
@@
 <pinref part="U1" gate="A" pin="PC5"/>
 <wire x1="264.16" y1="-76.454" x2="228.6" y2="-76.2" width="0.1524" layer="91"/>
-<junction x="264.16" y="-76.454"/>
-</segment>
-</net>
+</segment>
+</net>
