File: Schematic_Rev_3_Board_Rev_2/T17_Schematic_The_Useless_Box.sch (EAGLE design)
At the start: 18 parts, among them U1 ATMEGA328P-AU

Commit message: ACTUALLY updating the schematics this time. Picture added for modification on the wiki.
Parts:
- removed ARM_SERVO, LID_SERVO: (no value), con-lstb:MA03-1
- removed DC_MOTOR_1, DC_MOTOR_2: 22-23-2021, con-molex:22-23-2021
- removed ICSP: (no value), con-lstb:MA03-2
- removed MOTOR_DRIVER_1, MOTOR_DRIVER_2: BD6230F, rohm:BD6230F
- removed R3: 10k, rcl:R-EU_R0805
- removed S2: SWITCH-MOMENTARY-2SMD, SparkFun-Electromechanical:SWITCH-MOMENTARY-2SMD
- removed SCHMIDT_TRIGGER: ES2D, diode:ES2D
- added C5, C6, C7, C8, C9: 10nF, rcl:C-EUC0805
- added J1: AVR_SPI_PRG_6NS, SparkFun-Connectors:AVR_SPI_PRG_6NS
- added JP1, JP2: M02LOCK, SparkFun-Connectors:M02LOCK
- added JP3: ARM_SERVO, SparkFun-Connectors:M03PTH
- added JP4: LID_SERVO, SparkFun-Connectors:M03PTH
- added R1: 0, rcl:R-EU_R0805
- added S1: SWITCH-MOMENTARY-2SMD, SparkFun-Electromechanical:SWITCH-MOMENTARY-2SMD
- added TP1, TP10, TP11, TP12, TP13, TP2, TP3, TP4, TP5, TP6, TP7, TP8, TP9: TPB1,27, testpad:TPB1,27
- added U$1, U$2: LB1938FA-AH, microchip-MCP125x-xxx:LB1938FA-AH
- added U$3: INVERTING_SCHMITT_TRIGGER, SparkFun-DigitalIC:INVERTING_SCHMITT_TRIGGER
- R2: value 0 -> 10K
- U1: value ATMEGA328P-AU -> ATMEGA328P; device Atmel_By_element14_Batch_1-00:ATMEGA328P-AU -> SparkFun-DigitalIC:ATMEGA328_SMT
Connections:
- removed net +5V: ARM_SERVO.1, C1.1, IC1.OUT, ICSP.2, LID_SERVO.1, MOTOR_DRIVER_1.VCC@1, MOTOR_DRIVER_1.VCC@2, MOTOR_DRIVER_2.VCC@1, MOTOR_DRIVER_2.VCC@2, R3.2, U1.AVCC, U1.VCC, U1.VCC_2
- removed net N$19: MOTOR_DRIVER_1.RIN, U1.PC2
- removed net N$21: MOTOR_DRIVER_2.RIN, U1.PC4
- removed net N$22: LID_SERVO.2, U1.PC0
- removed net N$23: ARM_SERVO.2, U1.PC1
- removed net N$24: DC_MOTOR_2-1.S, MOTOR_DRIVER_2.OUT1
- removed net N$25: DC_MOTOR_1-1.S, MOTOR_DRIVER_1.OUT1
- removed net N$26: DC_MOTOR_1-2.S, MOTOR_DRIVER_1.OUT2
- removed net N$27: DC_MOTOR_2-2.S, MOTOR_DRIVER_2.OUT2
- new net 5V: C1.1, C3.2, C4.2, C5.2, C6.1, C7.1, C8.1, C9.1, IC1.OUT, J1.2, JP3.1, JP4.1, R2.2, TP2.TP, U$1.VCC, U$2.VCC, U$3.VCC, U1.AVCC, U1.VCC@1, U1.VCC@2
- new net N$10: JP4.2, TP3.TP, U1.PD3(INT1)
- new net N$13: TP5.TP, U$2.IN1, U1.PD6(AIN0)
- new net N$16: J1.5, R2.1, S1.2, U1.PC6(/RESET)
- new net N$2: JP1.1, TP9.TP, U$1.OUT1
- new net N$4: JP2.2, TP11.TP, U$2.OUT2
- new net N$5: JP2.1, TP10.TP, U$2.OUT1
- net GND: now also C3.1, C4.1, C5.1, C6.2, C7.2, C8.2, C9.2, J1.6, JP3.3, JP4.3, S1.1, U$1.P-GND, U$1.S-GND, U$2.P-GND, U$2.S-GND, U$3.GND, U1.AGND, U1.GND@1, U1.GND@2; no longer ARM_SERVO.3, C3.2, C4.2, ICSP.6, LID_SERVO.3, MOTOR_DRIVER_1.GND, S2.1, U1.GND, U1.GND_2, U1.GND_3
- net N$1: now also TP7.TP, U$1.IN1, U1.PB0(ICP); no longer ICSP.3, U1.PB5
- net N$11: now also R1.2, U$3.A; no longer C3.1, U1.PB6
- net N$12: now also G1.+, R1.1, TP1.TP; no longer ICSP.5, R3.1, S2.2, U1.PC6
- net N$14: now also J1.3, U1.PB5(SCK); no longer C4.1, U1.PB7
- net N$18: now also J1.1, U1.PB4(MISO); no longer MOTOR_DRIVER_1.FIN, U1.PC3
- net N$20: now also TP6.TP, U$2.IN2, U1.PD5(T1); no longer MOTOR_DRIVER_2.FIN, U1.PC5
- net N$3: now also JP1.2, TP12.TP, U$1.OUT2; no longer C2.1, IC1.IN, SCHMIDT_TRIGGER.C
- net N$6: now also TP8.TP, U$1.IN2, U1.PD7(AIN1); no longer R2.2, SCHMIDT_TRIGGER.A
- net N$7: now also J1.4, U1.PB3(MOSI/OC2); no longer G1.+, R2.1
- net N$8: now also JP3.2, TP4.TP, U1.PD4(XCK/T0); no longer ICSP.1, U1.PB4
- net N$9: now also C2.1, IC1.IN, TP13.TP, U$3.Y; no longer ICSP.4, U1.PB3
Other:
- note added: "3"
- note added: "9V-5V Power Supply"
- note added: "ICSP"
- note added: "Motor control block"
- note added: "Reset switch"
- note removed: "2"
- note removed: "ATMega328"
- note removed: "DC MOTORS"
- note removed: "MOTOR DRIVERS"
- note removed: "POWER SUPPLY"
- moved on the sheet: C1, C2, C3, C4, G1, IC1, R2

Commit message: Added mounting holes and ground plane staples
Parts:
- renumbered IC1 to 78L05
Changed lines of the file:
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@@
 <setting verticaltext="up"/>
 </settings>
-<grid distance="0.05" unitdist="inch" unit="inch" style="lines" multiple="1" display="yes" altdistance="0.01" altunitdist="inch" altunit="inch"/>
+<grid distance="0.1" unitdist="inch" unit="inch" style="lines" multiple="1" display="no" altdistance="0.01" altunitdist="inch" altunit="inch"/>
 <layers>
 <layer number="1" name="Top" color="4" fill="1" visible="no" active="no"/>
@@
 <part name="G1" library="battery" deviceset="AB9V" device=""/>
 <part name="U$3" library="SparkFun-DigitalIC" deviceset="INVERTING_SCHMITT_TRIGGER" device=""/>
-<part name="IC1" library="v-reg" deviceset="78LXX" device=""/>
+<part name="78L05" library="v-reg" deviceset="78LXX" device=""/>
 <part name="C1" library="rcl" deviceset="C-EU" device="C0805" value="10uF"/>
 <part name="C2" library="rcl" deviceset="C-EU" device="C0805" value="10uF"/>
@@
 <instance part="G1" gate="G$1" x="-82.55" y="223.52"/>
 <instance part="U$3" gate="G$1" x="-29.21" y="223.52"/>
-<instance part="IC1" gate="1" x="21.59" y="226.06"/>
+<instance part="78L05" gate="1" x="21.59" y="226.06"/>
 <instance part="C1" gate="G$1" x="39.37" y="215.9"/>
 <instance part="C2" gate="G$1" x="6.35" y="215.9"/>
@@
 </segment>
 <segment>
-<pinref part="IC1" gate="1" pin="GND"/>
+<pinref part="78L05" gate="1" pin="GND"/>
 <pinref part="GND3" gate="1" pin="GND"/>
 <wire x1="21.59" y1="218.44" x2="21.59" y2="208.28" width="0.1524" layer="91"/>
@@
 <wire x1="6.35" y1="218.44" x2="6.35" y2="226.06" width="0.1524" layer="91"/>
 <junction x="6.35" y="218.44"/>
-<pinref part="IC1" gate="1" pin="IN"/>
+<pinref part="78L05" gate="1" pin="IN"/>
 <wire x1="6.35" y1="226.06" x2="13.97" y2="226.06" width="0.1524" layer="91"/>
 <pinref part="C2" gate="G$1" pin="1"/>
@@
 </segment>
 <segment>
-<pinref part="IC1" gate="1" pin="OUT"/>
+<pinref part="78L05" gate="1" pin="OUT"/>
 <wire x1="29.21" y1="226.06" x2="39.37" y2="226.06" width="0.1524" layer="91"/>
 <pinref part="C1" gate="G$1" pin="1"/>

Commit message: submittable board?
Parts:
- removed 78L05: (no value), v-reg:78LXX
- removed G1: AB9V, battery:AB9V
- removed TP13: TPB1,27, testpad:TPB1,27
- removed U$3: INVERTING_SCHMITT_TRIGGER, SparkFun-DigitalIC:INVERTING_SCHMITT_TRIGGER
- added 9V-BATTERY-CLIP: M02LOCK, SparkFun-Connectors:M02LOCK
- added C10, C11: 22pF, rcl:C-EUC0805
- added IC1: (no value), SparkFun-PowerIC:V_REG_78XX-TO-220
- added JP5: (no value), SparkFun-Connectors:M06NO_SILK_FEMALE_PTH
- added Q1: 16kHz, special:XTAL/S
- added R3, R4, R5, R6: 10K, rcl:R-EU_R0805
- C6, C7: value 10nF -> 10uF
Connections:
- new net N$15: JP5.4, U1.PD1(TXD)
- new net N$17: C11.2, Q1.1, U1.PB7(XTAL2/TOSC2)
- new net N$19: C10.2, Q1.2, U1.PB6(XTAL1/TOSC1)
- net 5V: now also IC1.OUT, JP3.2, JP4.2; no longer 78L05.OUT, JP3.1, JP4.1, U$3.VCC
- net GND: now also 9V-BATTERY-CLIP.1, C10.1, C11.1, IC1.GND, JP5.1, R3.1, R4.1, R5.1, R6.1; no longer 78L05.GND, G1.-, U$3.GND
- net N$1: now also R6.2
- net N$10: now also JP4.1; no longer JP4.2
- net N$11: now also C2.1, IC1.IN; no longer U$3.A
- net N$12: now also 9V-BATTERY-CLIP.2; no longer G1.+
- net N$13: now also R3.2
- net N$20: now also R4.2
- net N$6: now also R5.2
- net N$8: now also JP3.1; no longer JP3.2
- net N$9: now also JP5.5, U1.PD0(RXD); no longer 78L05.IN, C2.1, TP13.TP, U$3.Y
Other:
- note added: "3.5"
- note removed: "3"
- moved on the sheet: C1, C5, TP2, TP5

Commit message: Adding the final ckt design
Parts:
- added C12: 10nF, rcl:C-EUC0805
- added TOGGLE: M02LOCK, SparkFun-Connectors:M02LOCK
- Q1: value 16kHz -> 16MHz
- renumbered JP1 to R-MOTOR, JP2 to L-MOTOR, JP5 to PROGRAMMING
Connections:
- new net N$21: TOGGLE.2, U1.PC1(ADC1)
- net 5V: now also C12.1, TOGGLE.1
- net GND: now also C12.2
Changed lines of the file:
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@@
 <part name="U1" library="SparkFun-DigitalIC" deviceset="ATMEGA328_SMT" device="" value="ATMEGA328P"/>
 <part name="J1" library="SparkFun-Connectors" deviceset="AVR_SPI_PRG_6" device="NS"/>
-<part name="JP1" library="SparkFun-Connectors" deviceset="M02" device="LOCK"/>
-<part name="JP2" library="SparkFun-Connectors" deviceset="M02" device="LOCK"/>
+<part name="R-MOTOR" library="SparkFun-Connectors" deviceset="M02" device="LOCK"/>
+<part name="L-MOTOR" library="SparkFun-Connectors" deviceset="M02" device="LOCK"/>
 <part name="JP3" library="SparkFun-Connectors" deviceset="M03" device="PTH" value="ARM_SERVO"/>
 <part name="JP4" library="SparkFun-Connectors" deviceset="M03" device="PTH" value="LID_SERVO"/>
@@
 <part name="TP2" library="testpad" deviceset="TP" device="B1,27"/>
 <part name="9V-BATTERY-CLIP" library="SparkFun-Connectors" deviceset="M02" device="LOCK"/>
-<part name="Q1" library="special" deviceset="XTAL/S" device="" value="16kHz"/>
+<part name="Q1" library="special" deviceset="XTAL/S" device="" value="16MHz"/>
 <part name="C10" library="rcl" deviceset="C-EU" device="C0805" value="22pF"/>
 <part name="C11" library="rcl" deviceset="C-EU" device="C0805" value="22pF"/>
 <part name="GND11" library="supply1" deviceset="GND" device=""/>
 <part name="GND26" library="supply1" deviceset="GND" device=""/>
-<part name="JP5" library="SparkFun-Connectors" deviceset="M06" device="NO_SILK_FEMALE_PTH"/>
+<part name="PROGRAMMING" library="SparkFun-Connectors" deviceset="M06" device="NO_SILK_FEMALE_PTH"/>
 <part name="GND27" library="supply1" deviceset="GND" device=""/>
 <part name="IC1" library="SparkFun-PowerIC" deviceset="V_REG_78XX" device="-TO-220"/>
+<part name="TOGGLE" library="SparkFun-Connectors" deviceset="M02" device="LOCK"/>
+<part name="SUPPLY7" library="SparkFun-Aesthetics" deviceset="5V" device=""/>
+<part name="C12" library="rcl" deviceset="C-EU" device="C0805" value="10nF"/>
+<part name="GND28" library="supply1" deviceset="GND" device=""/>
 </parts>
 <sheets>
@@
 <instance part="U1" gate="G$1" x="86.36" y="101.6"/>
 <instance part="J1" gate="G$1" x="83.82" y="24.13" rot="R270"/>
-<instance part="JP1" gate="G$1" x="223.52" y="43.18" rot="R180"/>
-<instance part="JP2" gate="G$1" x="222.25" y="83.82" rot="R180"/>
+<instance part="R-MOTOR" gate="G$1" x="223.52" y="43.18" rot="R180"/>
+<instance part="L-MOTOR" gate="G$1" x="222.25" y="83.82" rot="R180"/>
 <instance part="JP3" gate="G$1" x="226.06" y="162.56" rot="R180"/>
 <instance part="JP4" gate="G$1" x="226.06" y="190.5" rot="R180"/>
@@
 <instance part="GND11" gate="1" x="1.27" y="101.6"/>
 <instance part="GND26" gate="1" x="1.27" y="88.9"/>
-<instance part="JP5" gate="G$1" x="90.678" y="162.052" rot="R270"/>
+<instance part="PROGRAMMING" gate="G$1" x="90.678" y="162.052" rot="R270"/>
 <instance part="GND27" gate="1" x="76.454" y="149.098"/>
 <instance part="IC1" gate="G$1" x="21.59" y="226.06"/>
+<instance part="TOGGLE" gate="G$1" x="166.37" y="142.24" rot="R180"/>
+<instance part="SUPPLY7" gate="G$1" x="154.432" y="156.464"/>
+<instance part="C12" gate="G$1" x="151.892" y="150.114" rot="R270"/>
+<instance part="GND28" gate="1" x="136.652" y="147.574"/>
 </instances>
 <busses>
@@
 </segment>
 <segment>
-<pinref part="JP5" gate="G$1" pin="1"/>
+<pinref part="PROGRAMMING" gate="G$1" pin="1"/>
 <wire x1="85.598" y1="156.972" x2="76.454" y2="156.972" width="0.1524" layer="91"/>
 <wire x1="76.454" y1="156.972" x2="76.454" y2="151.638" width="0.1524" layer="91"/>
 <pinref part="GND27" gate="1" pin="GND"/>
 </segment>
+<segment>
+<pinref part="C12" gate="G$1" pin="2"/>
+<wire x1="146.812" y1="150.114" x2="136.652" y2="150.114" width="0.1524" layer="91"/>
+<pinref part="GND28" gate="1" pin="GND"/>
+</segment>
 </net>
 <net name="N$2" class="0">
@@
 <wire x1="181.61" y1="46.99" x2="201.93" y2="46.99" width="0.1524" layer="91"/>
 <wire x1="201.93" y1="46.99" x2="201.93" y2="43.18" width="0.1524" layer="91"/>
-<pinref part="JP1" gate="G$1" pin="1"/>
+<pinref part="R-MOTOR" gate="G$1" pin="1"/>
 <wire x1="201.93" y1="43.18" x2="215.9" y2="43.18" width="0.1524" layer="91"/>
 <pinref part="TP9" gate="G$1" pin="TP"/>
@@
 <wire x1="181.61" y1="39.37" x2="201.93" y2="39.37" width="0.1524" layer="91"/>
 <wire x1="201.93" y1="39.37" x2="201.93" y2="40.64" width="0.1524" layer="91"/>
-<pinref part="JP1" gate="G$1" pin="2"/>
+<pinref part="R-MOTOR" gate="G$1" pin="2"/>
 <wire x1="201.93" y1="40.64" x2="215.9" y2="40.64" width="0.1524" layer="91"/>
 <pinref part="TP12" gate="G$1" pin="TP"/>
@@
 <wire x1="181.61" y1="80.01" x2="195.58" y2="80.01" width="0.1524" layer="91"/>
 <wire x1="195.58" y1="80.01" x2="195.58" y2="81.28" width="0.1524" layer="91"/>
-<pinref part="JP2" gate="G$1" pin="2"/>
+<pinref part="L-MOTOR" gate="G$1" pin="2"/>
 <wire x1="195.58" y1="81.28" x2="214.63" y2="81.28" width="0.1524" layer="91"/>
 <pinref part="TP11" gate="G$1" pin="TP"/>
@@
 <wire x1="195.58" y1="87.63" x2="195.58" y2="83.82" width="0.1524" layer="91"/>
 <wire x1="195.58" y1="83.82" x2="214.63" y2="83.82" width="0.1524" layer="91"/>
-<pinref part="JP2" gate="G$1" pin="1"/>
+<pinref part="L-MOTOR" gate="G$1" pin="1"/>
 <wire x1="214.63" y1="83.82" x2="215.9" y2="83.82" width="0.1524" layer="91"/>
 <junction x="214.63" y="83.82"/>
@@
 <wire x1="218.44" y1="190.5" x2="201.93" y2="190.5" width="0.1524" layer="91"/>
 <wire x1="201.93" y1="190.5" x2="201.93" y2="193.04" width="0.1524" layer="91"/>
+</segment>
+<segment>
+<pinref part="C12" gate="G$1" pin="1"/>
+<wire x1="154.432" y1="142.24" x2="154.432" y2="150.114" width="0.1524" layer="91"/>
+<pinref part="SUPPLY7" gate="G$1" pin="5V"/>
+<wire x1="154.432" y1="150.114" x2="154.432" y2="156.464" width="0.1524" layer="91"/>
+<junction x="154.432" y="150.114"/>
+<pinref part="TOGGLE" gate="G$1" pin="1"/>
+<wire x1="158.75" y1="142.24" x2="154.432" y2="142.24" width="0.1524" layer="91"/>
 </segment>
 </net>
@@
 <wire x1="111.76" y1="104.14" x2="114.3" y2="104.14" width="0.1524" layer="91"/>
 <wire x1="114.3" y1="104.14" x2="114.3" y2="151.638" width="0.1524" layer="91"/>
-<pinref part="JP5" gate="G$1" pin="5"/>
+<pinref part="PROGRAMMING" gate="G$1" pin="5"/>
 <wire x1="114.3" y1="151.638" x2="95.758" y2="151.638" width="0.1524" layer="91"/>
 <wire x1="95.758" y1="151.638" x2="95.758" y2="156.972" width="0.1524" layer="91"/>
@@
 <wire x1="111.76" y1="101.6" x2="116.84" y2="101.6" width="0.1524" layer="91"/>
 <wire x1="116.84" y1="101.6" x2="116.84" y2="142.24" width="0.1524" layer="91"/>
-<pinref part="JP5" gate="G$1" pin="4"/>
+<pinref part="PROGRAMMING" gate="G$1" pin="4"/>
 <wire x1="116.84" y1="142.24" x2="93.218" y2="142.24" width="0.1524" layer="91"/>
 <wire x1="93.218" y1="142.24" x2="93.218" y2="156.972" width="0.1524" layer="91"/>
 </segment>
 </net>
+<net name="N$21" class="0">
+<segment>
+<pinref part="U1" gate="G$1" pin="PC1(ADC1)"/>
+<pinref part="TOGGLE" gate="G$1" pin="2"/>
+<wire x1="111.76" y1="124.46" x2="158.75" y2="124.46" width="0.1524" layer="91"/>
+<wire x1="158.75" y1="124.46" x2="158.75" y2="139.7" width="0.1524" layer="91"/>
+</segment>
+</net>
